File: Hardware/ZED-F9P_NEO-D9S_Combo.brd (EAGLE design)
At the start: 43.2 x 63.5 mm, 179 parts, among them J1 ANTENNA-SMA-GROUNDEDEDGE_SMA, J2 Qwiic Right Angle, J4 Qwiic Right Angle, U1 U-BLOX_NEO-D9S-00B, U2 3.3V, U4 U-BLOX_ZED-F9P, U5 ESD Diode, U6 ESD Diode, U7 BP2G1+_POWER_SPLITTER

Commit message: Adds new panel - bottom silk change
Parts:
- moved U$80 0.25 mm to (6.60, 51.2)
- moved U$82 0.25 mm to (6.60, 56.8)
- moved U$76 0.25 mm to (9.14, 53.3)
- moved U$79 0.25 mm to (7.87, 51.1)
- moved U$81 0.25 mm to (7.87, 56.8)
Changed lines of the file:
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@@
 <layer number="19" name="Unrouted" color="6" fill="1" visible="yes" active="yes"/>
 <layer number="20" name="Dimension" color="15" fill="1" visible="yes" active="yes"/>
-<layer number="21" name="tPlace" color="16" fill="1" visible="no" active="yes"/>
-<layer number="22" name="bPlace" color="14" fill="1" visible="no" active="yes"/>
+<layer number="21" name="tPlace" color="16" fill="1" visible="yes" active="yes"/>
+<layer number="22" name="bPlace" color="14" fill="1" visible="yes" active="yes"/>
 <layer number="23" name="tOrigins" color="15" fill="1" visible="yes" active="yes"/>
 <layer number="24" name="bOrigins" color="15" fill="1" visible="yes" active="yes"/>
@@
 <element name="U$73" library="top" package="OPEN_JUMPERS13" value="" x="22.225" y="50.927" smashed="yes" rot="MR90"/>
 <element name="U$74" library="top" package="TO_ISOLATE_UART214" value="" x="20.828" y="50.927" smashed="yes" rot="MR90"/>
-<element name="U$76" library="top" package="DEF_ADDRESS#_12" value="" x="8.89" y="53.34" smashed="yes" rot="MR90"/>
-<element name="U$79" library="top" package="NEO#D9S#13" value="" x="7.62" y="51.054" smashed="yes" rot="MR90"/>
-<element name="U$80" library="top" package="ZED#F9P#13" value="" x="6.35" y="51.181" smashed="yes" rot="MR90"/>
-<element name="U$81" library="top" package="0X4313" value="" x="7.62" y="56.769" smashed="yes" rot="MR90"/>
-<element name="U$82" library="top" package="0X4213" value="" x="6.35" y="56.769" smashed="yes" rot="MR90"/>
+<element name="U$76" library="top" package="DEF_ADDRESS#_12" value="" x="9.144" y="53.34" smashed="yes" rot="MR90"/>
+<element name="U$79" library="top" package="NEO#D9S#13" value="" x="7.874" y="51.054" smashed="yes" rot="MR90"/>
+<element name="U$80" library="top" package="ZED#F9P#13" value="" x="6.604" y="51.181" smashed="yes" rot="MR90"/>
+<element name="U$81" library="top" package="0X4313" value="" x="7.874" y="56.769" smashed="yes" rot="MR90"/>
+<element name="U$82" library="top" package="0X4213" value="" x="6.604" y="56.769" smashed="yes" rot="MR90"/>
 <element name="LOGO6" library="SparkFun-Aesthetics" package="QWIIC_5MM" value="QWIIC_LOGO_5MM" x="8.89" y="56.769" smashed="yes"/>
 </elements>
